File: PCB/Analog_Macropad_v02/Power.kicad_sch (KiCad schematic)
At the start: 1 part

Commit message: lots of modifs
Parts:
- added C14, C15: 1uF, symbol Device:C
- added C16, C17: 4.7uF, symbol Device:C
- added C18: 0.1uF, symbol Device:C
- added D1: LED, symbol Device:LED
- added R5: TBD, symbol Device:R
- added R6: 470R, symbol Device:R
- added R7: 330R, symbol Device:R
- added R8: 2k2, symbol Device:R
- added SW2: JS202011JAQN, JS202011JAQN_CNK, symbol Analog_Macropad_v02:JS202011JAQN
- added U3: 3.3V Regulator, DBV0005A_N, symbol Analog_Macropad_v02:3.3V Regulator
- added U4: Li-Ion Charger, SOT-23-5_MC_MCH, symbol Analog_Macropad_v02:Li-Ion Charger
- added U5: Battery Protection, DSE0006A, symbol Analog_Macropad_v02:Battery Protection
- added U6: Dual NMOSFET, SOT-363 US6_TOS, symbol Analog_Macropad_v02:Dual NMOSFET
Connections:
- net +VBAT: now reaches BT1.1 (+)
- net +VBAT: now also R7.1, SW2.6
- net at BT1.2 (-): now also C18.2, U5.4 (VSS), U6.4 (S2)
- new net: C18.1, R7.2, U5.5 (BAT)
- new net: R5.1, U4.5 (PROG)
- new net: U5.2 (COUT), U6.2 (G1)
- new net: U6.3 (D2), U6.6 (D1)
- new net: U5.3 (DOUT), U6.5 (G2)
- new net: SW2.3, SW2.7
- new net: D1.1 (K), R6.1
- new net: R6.2, U4.1 (STAT)
- new net: R8.1, U5.6 (V-)
- new net 3V3: C15.1, U3.5 (OUT)
- new net ChargerOut: C17.1, SW2.5, U4.3 (VBAT)
- new net GND: C14.2, C15.2, C16.2, C17.2, R5.2, R8.2, U3.2 (GND), U4.2 (VSS), U6.1 (S1)
- new net RegIn: C14.1, SW2.2, U3.1 (IN), U3.3 (EN)
- new net VBUS: C16.1, D1.2 (A), SW2.1, U4.4 (VDD)
- no-connect marks 0 -> 2
Other:
- note added: "Battery Charging"
- note added: "Battery Protection"
- note added: "Bluetooth Toggle"
- note added: "Voltage Regulation"
- company: (none) -> Jean-Christophe Gauthier
- moved on the sheet: BT1
